Commit message: Updated URDF files

File: cobot_description/robots/cobot_navigation.urdf.xacro (robot description, xacro)
@@ -7,3 +7,4 @@
  <cobot_top parent_link="frame_right_top_link" height_offset="${frame_top_length}" />
  <kinect parent_link="top_link" parent_x="-0.25 " parent_y="0.75" parent_z="0" parent_ox="${pi/2.0}" parent_oy="${pi/2.0}" parent_oz="${pi/2.0}" />
+ <ultrasoon parent_link="platform_link" panel="front" side="middle" parent_x="-0.4 " parent_y="0.75" parent_z="0" parent_ox="0" parent_oy="0" parent_oz="0" />
 </robot>

File: cobot_description/urdf/cobot_library.urdf.xacro (robot description, xacro)
@@ -4,14 +4,50 @@
  -->
 <robot name="library" xmlns:xacro="http://ros.org/wiki/xacro">
-  <!-- Materials -->
+  <!-- ### Materials ### -->
+  <!--
+    Material constants of the robot(like colors)
+  -->
   <xacro:include filename="$(find cobot_description)/urdf/materials/materials.urdf.xacro"/>
-  <!-- Platform -->
+  <!-- ### Platform ### -->
+  <!--
+    Base (Platform) of the robot
+  -->
   <xacro:include filename="$(find cobot_description)/urdf/platform/base.urdf.xacro"/>
+  <!--
+    Body of the robot
+    @param parent_link name of the parent link
+    @param platform_height z-distance of the platform where the body is atached to
+  -->
   <xacro:include filename="$(find cobot_description)/urdf/platform/body.urdf.xacro"/>
+  <!--
+    Top part of the robot
+    @param parent_link name of the parent link
+    @param height_offset z-distance relative to the parent link
+  -->
   <xacro:include filename="$(find cobot_description)/urdf/platform/top.urdf.xacro"/>
-  <!-- Sensors -->
+  <!-- ### Sensors ### -->
+  <!--
+    Kinect
+    @param parent_link name of the parent link
+    @param parent_x x-coordinate relative to the parent link
+    @param parent_y y-coordinate relative to the parent link
+    @param parent_z z-coordinate relative to the parent link
+    @param parent_ox x-axis turning relative to the parent link
+    @param parent_oy y-axis turning relative to the parent link
+    @param parent_oz z-axis turning relative to the parent link
+  -->
   <xacro:include filename="$(find cobot_description)/urdf/sensors/kinect.urdf.xacro"/>
-<!--
+  <!--
+    Ultrasoon
+    @param parent_link name of the parent link
+    @param panel panel where the sensor is attached to (e.g. front,back,left_side,right_side)
+    @param side the place on the panel (e.g. left,middle,right)
+    @param parent_x x-coordinate relative to the parent link
+    @param parent_y y-coordinate relative to the parent link
+    @param parent_z z-coordinate relative to the parent link
+    @param parent_ox x-axis turning relative to the parent link
+    @param parent_oy y-axis turning relative to the parent link
+    @param parent_oz z-axis turning relative to the parent link
+  -->
   <xacro:include filename="$(find cobot_description)/urdf/sensors/ultrasoon.urdf.xacro"/>
--->
 </robot>

File: cobot_description/urdf/sensors/ultrasoon.urdf.xacro (robot description, xacro)
@@ -14,5 +14,5 @@
       <parent link="${parent_link}" />
       <child link="ultrasoon_${panel}_${side}_link" />
-      <origin xyz="${parent_x} ${parent_y} ${parent_z" rpy="${parent_ox} ${parent_oy} ${parent_oz}" />
+      <origin xyz="${parent_x} ${parent_y} ${parent_z}" rpy="${parent_ox} ${parent_oy} ${parent_oz}" />
     </joint>
   </xacro:macro>
