Commit message: Rotated model, robot faces now in +x direction, for more consistency

File: cobot_description/robots/cobot_threemxl_manual.urdf.xacro (robot description, xacro)
@@ -4,6 +4,7 @@
  <xacro:include filename="$(find cobot_description)/urdf/constants.urdf.xacro" />
  <cobot_base />
+<!--
  <cobot_body parent_link="platform_link" platform_height="${platform_height}"/>
  <cobot_top parent_link="frame_right_top_link" height_offset="${frame_top_length}" />
- <kinect parent_link="base_link" parent_x="0 " parent_y="0.10" parent_z="0.35" parent_ox="0" parent_oy="0" parent_oz="0" />
+-->
 </robot>

File: cobot_description/robots/cobot_threemxl_navigation.urdf.xacro (robot description, xacro)
@@ -4,7 +4,7 @@
  <xacro:include filename="$(find cobot_description)/urdf/constants.urdf.xacro" />
  <cobot_base />
- <cobot_body parent_link="platform_link" platform_height="${platform_height}"/>
+ <cobot_body parent_link="platform_link"/>
  <cobot_top parent_link="frame_right_top_link" height_offset="${frame_top_length}" />
- <kinect parent_link="top_link" parent_x="-0.25 " parent_y="0.75" parent_z="0" parent_ox="${pi/2.0}" parent_oy="${pi/2.0}" parent_oz="${pi/2.0}" />
- <ultrasoon parent_link="platform_link" panel="front" side="middle" parent_x="-0.4 " parent_y="0.75" parent_z="0" parent_ox="0" parent_oy="0" parent_oz="0" />
+ <kinect parent_link="top_link" parent_x="0.75 " parent_y="0.25" parent_z="0" parent_ox="${pi}" parent_oy="0" parent_oz="0" />
+ <ultrasoon parent_link="platform_link" panel="front" side="middle" parent_x="0.57" parent_y="0.23" parent_z="0" parent_ox="0" parent_oy="0" parent_oz="0" />
 </robot>

File: cobot_description/urdf/cobot_library.urdf.xacro (robot description, xacro)
@@ -17,5 +17,4 @@
     Body of the robot
     @param parent_link name of the parent link
-    @param platform_height z-distance of the platform where the body is atached to
   -->
   <xacro:include filename="$(find cobot_description)/urdf/platform/body.urdf.xacro"/>

File: cobot_description/urdf/platform/base.urdf.xacro (robot description, xacro)
@@ -4,8 +4,8 @@
   <xacro:macro name="cobot_base">
     <xacro:base_platform />
-    <xacro:powered_wheel parent_link="base_link" side="left" mirror="-1" />
-    <xacro:powered_wheel parent_link="base_link" side="right" mirror="1" />
-    <xacro:caster_wheel parent_link="base_link" side="left" mirror="-1" />
-    <xacro:caster_wheel parent_link="base_link" side="right" mirror="1" />
+    <xacro:powered_wheel parent_link="base_link" side="left" mirror="1" />
+    <xacro:powered_wheel parent_link="base_link" side="right" mirror="-1" />
+    <xacro:caster_wheel parent_link="base_link" side="left" mirror="1" />
+    <xacro:caster_wheel parent_link="base_link" side="right" mirror="-1" />
   </xacro:macro>
   <xacro:include filename="$(find cobot_description)/urdf/constants.urdf.xacro" />
@@ -22,5 +22,5 @@
       <link name="powered_${side}_wheel_link">
         <visual>
-          <origin xyz="0 0 0" rpy="${pi/2} 0 ${pi/2}" />
+          <origin xyz="0 0 0" rpy="${pi/2} 0 0" />
           <geometry>
             <cylinder radius="${powered_wheel_diameter/2.0}" length="${powered_wheel_thickness}"/>
@@ -35,5 +35,5 @@
         <parent link="${parent_link}"/>
         <child link="powered_${side}_wheel_link"/>
-        <origin xyz="${(platform_width/2.0)*mirror+powered_wheel_spacing} 0 0" rpy="0 0 0"/>
+        <origin xyz="0 ${(platform_width/2.0)*mirror+powered_wheel_spacing} 0" rpy="0 0 0"/>
       </joint>
     </xacro:macro>
@@ -41,5 +41,5 @@
       <link name="caster_${side}_wheel_link">
         <visual>
-          <origin xyz="0 0 0" rpy="${pi/2} 0 ${pi/2}" />
+          <origin xyz="0 0 0" rpy="${pi/2} 0 0" />
           <geometry>
             <cylinder radius="${caster_wheel_diameter/2.0}" length="${caster_wheel_thickness}"/>
@@ -54,5 +54,5 @@
         <parent link="${parent_link}"/>
         <child link="caster_${side}_wheel_link"/>
-        <origin xyz="${(platform_width/2.0)*mirror} ${-platform_length+center_wheel_axis_to_front_platform_distance} -${(powered_wheel_diameter/2.0)-(caster_wheel_diameter/2.0)}" rpy="0 0 0"/>
+        <origin xyz="${-platform_length+center_wheel_axis_to_front_platform_distance} ${(platform_width/2.0)*mirror} -${(powered_wheel_diameter/2.0)-(caster_wheel_diameter/2.0)}" rpy="0 0 0"/>
       </joint>
     </xacro:macro>
@@ -74,5 +74,5 @@
       <origin xyz="0 0 0" rpy="0 0 0" />
         <geometry>
-          <box size="${platform_width} .02 0.01" />
+          <box size=".02 ${platform_width} 0.01" />
         </geometry>
       </visual>
@@ -80,7 +80,7 @@
     <link name="platform_link">
       <visual>
-      <origin xyz="-${platform_width/2.0} ${platform_length/2.0} 0" rpy="0 0 0" />
+      <origin xyz="${platform_length/2.0} ${platform_width/2.0} -${platform_height/2.0}" rpy="0 0 0" />
         <geometry>
-          <box size="${platform_width} ${platform_length} ${platform_height}" />
+          <box size="${platform_length} ${platform_width} ${platform_height}" />
         </geometry>
           <material name="light_grey" />
@@ -97,5 +97,5 @@
       <parent link="base_link" />
       <child link="platform_link" />
-      <origin xyz="${platform_width/2.0} ${-platform_length+center_wheel_axis_to_front_platform_distance} 0" rpy="0 0 0" />
+      <origin xyz="${-platform_length+center_wheel_axis_to_front_platform_distance} -${platform_width/2.0} ${platform_height/2.0}" rpy="0 0 0" />
     </joint>
   </xacro:macro>

File: cobot_description/urdf/platform/body.urdf.xacro (robot description, xacro)
@@ -1,8 +1,8 @@
 <?xml version="1.0"?>
 <robot name="cobot_body" xmlns:xacro="http://ros.org/wiki/xacro">
-  <xacro:macro name="cobot_body" params="parent_link platform_height" >
+  <xacro:macro name="cobot_body" params="parent_link" >
     <xacro:body />
-    <xacro:frame_top parent_link="body_link" side="left" from_body="-0.46" />
-    <xacro:frame_top parent_link="body_link" side="right" from_body="0" />
+    <xacro:frame_top parent_link="body_link" side="left" mirror="1"/>
+    <xacro:frame_top parent_link="body_link" side="right" mirror="0"/>
   </xacro:macro>
   <xacro:include filename="$(find cobot_description)/urdf/constants.urdf.xacro" />
@@ -11,5 +11,6 @@
   <!-- taken from mesh file -->
   <xacro:property name="body_height" value="0.74" />
-  <xacro:macro name="frame_top" params="parent_link side from_body">
+  <xacro:property name="body_width" value="0.46" />
+  <xacro:macro name="frame_top" params="parent_link side mirror">
     <link name="frame_${side}_top_link">
      <visual>
@@ -24,11 +25,11 @@
       <parent link="${parent_link}" />
       <child link="frame_${side}_top_link" />
-      <origin xyz="${from_body} 0 ${body_height}" rpy="0 0 0" />
+      <origin xyz="0 ${body_width*mirror} ${body_height}" rpy="0 0 0" />
     </joint>
   </xacro:macro>
-  <xacro:macro name="body" param="parent_link ,platform_height">
+  <xacro:macro name="body" param="parent_link">
    <link name="body_link">
       <visual>
-      <origin xyz="0 0 0" rpy="0 0 ${pi/2}" />
+      <origin xyz="0 0 0" rpy="0 0 0" />
        <geometry>
          <mesh filename="package://cobot_description/meshes/dae/body.dae" />
@@ -39,5 +40,5 @@
       <parent link="${parent_link}" />
       <child link="body_link" />
-      <origin xyz="0 0 ${platform_height/2.0}" rpy="0 0 0" />
+      <origin xyz="0 0 0" rpy="0 0 0" />
     </joint>
   </xacro:macro>

File: cobot_description/urdf/platform/top.urdf.xacro (robot description, xacro)
@@ -8,5 +8,5 @@
     <link name="top_link">
        <visual>
-       <origin xyz="0 0 0" rpy="0 0 ${pi/2.0}" />
+       <origin xyz="0 0 0" rpy="0 0 0" />
         <geometry>
           <mesh filename="package://cobot_description/meshes/dae/top.dae" />

File: cobot_description/urdf/sensors/kinect.urdf.xacro (robot description, xacro)
@@ -9,5 +9,5 @@
   <link name="camera_rgb_frame">
      <visual>
-     <origin xyz="0 0.15 0" rpy="${parent_ox + pi/2.0} ${parent_oy} ${parent_oz}" />
+     <origin xyz="0.15 0 0" rpy="${parent_ox} ${parent_oy + pi/2} ${parent_oz}" />
       <geometry>
         <cylinder radius="${camera_diameter_lens/2.0}" length="0.3" />
@@ -18,5 +18,5 @@
   <link name="camera_rgb_optical_frame">
      <visual>
-     <origin xyz="0 0.15 0" rpy="${parent_ox + pi/2.0} ${parent_oy} ${parent_oz}" />
+     <origin xyz="0.15 0 0" rpy="${parent_ox} ${parent_oy + pi/2} ${parent_oz}" />
       <geometry>
         <cylinder radius="${camera_diameter_lens/4.0}" length="0.3" />
@@ -29,5 +29,5 @@
     <origin xyz="0 0 0" rpy="0 0 0"/>
      <geometry>
-       <box size="${camera_length} ${camera_width} ${camera_height}" />
+       <box size="${camera_width} ${camera_length} ${camera_height}" />
      </geometry>
     <material name="green" />
@@ -36,5 +36,5 @@
 	<link name="camera_depth_frame">
    <visual>
-     <origin xyz="0 0.15 0" rpy="${parent_ox + pi/2.0} ${parent_oy} ${parent_oz}" />
+     <origin xyz="0.15 0 0" rpy="${parent_ox} ${parent_oy + pi/2.0} ${parent_oz}" />
       <geometry>
         <cylinder radius="${camera_diameter_lens/2.0}" length="0.3" />
@@ -45,5 +45,5 @@
 	<link name="camera_depth_optical_frame">
    <visual>
-     <origin xyz="0 0.15 0" rpy="${parent_ox + pi/2.0} ${parent_oy} ${parent_oz}" />
+     <origin xyz="0.15 0 0" rpy="${parent_ox} ${parent_oy + pi/2.0} ${parent_oz}" />
       <geometry>
         <cylinder radius="${camera_diameter_lens/4.0}" length="0.3" />
@@ -63,10 +63,10 @@
    </joint>
    <joint name="camera_joint" type="fixed">
-     <origin xyz="0.007 0 0" rpy="0 0 0"/>
+     <origin xyz="0 0.0125 0" rpy="0 0 0"/>
      <parent link="camera_rgb_frame"/>
      <child link="camera_link"/>
    </joint>
 	<joint name="camera_depth_joint" type="fixed">
-	  <origin xyz="0.025 0 0" rpy="0 0 0" />
+	  <origin xyz="0 0.027 0" rpy="0 0 0" />
 	  <parent link="camera_rgb_frame" />
 	  <child link="camera_depth_frame" />
