Commit message: Added ultrasoon (example)

File: cobot_description/robots/cobot_threemxl_navigation.urdf.xacro (robot description, xacro)
@@ -6,5 +6,12 @@
  <cobot_body parent_link="platform_link"/>
  <cobot_top parent_link="frame_right_top_link" height_offset="${frame_top_length}" />
- <kinect parent_link="top_link" parent_x="0.75 " parent_y="0.25" parent_z="0" parent_ox="${pi}" parent_oy="0" parent_oz="0" />
- <ultrasoon parent_link="platform_link" panel="front" side="middle" parent_x="0.57" parent_y="0.23" parent_z="0" parent_ox="0" parent_oy="0" parent_oz="0" />
+ <kinect parent_link="base_link" parent_x="0.1 " parent_y="0" parent_z="1.0" parent_ox="${pi}" parent_oy="0" parent_oz="0" />
+ <ultrasoon parent_link="base_link" panel="front" side="middle" parent_x="0.10" parent_y="0" parent_z="0" parent_ox="0" parent_oy="0" parent_oz="0" />
+ <ultrasoon parent_link="base_link" panel="front" side="left" parent_x="0.10" parent_y="-0.15" parent_z="0" parent_ox="0" parent_oy="0" parent_oz="0" />
+ <ultrasoon parent_link="base_link" panel="front" side="right" parent_x="0.10" parent_y="0.15" parent_z="0" parent_ox="0" parent_oy="0" parent_oz="0" />
+ <ultrasoon parent_link="base_link" panel="back" side="middle" parent_x="-0.47" parent_y="0" parent_z="0" parent_ox="0" parent_oy="0" parent_oz="${pi}" />
+ <ultrasoon parent_link="base_link" panel="back" side="left" parent_x="-0.47" parent_y="-0.15" parent_z="0" parent_ox="0" parent_oy="0" parent_oz="${pi}" />
+ <ultrasoon parent_link="base_link" panel="back" side="right" parent_x="-0.47" parent_y="0.15" parent_z="0" parent_ox="0" parent_oy="0" parent_oz="${pi}" />
+ <ultrasoon parent_link="base_link" panel="left" side="left" parent_x="-0.3" parent_y="0.23" parent_z="0" parent_ox="0" parent_oy="0" parent_oz="${pi/2}" />
+ <ultrasoon parent_link="base_link" panel="right" side="right" parent_x="-0.3" parent_y="-0.23" parent_z="0" parent_ox="0" parent_oy="0" parent_oz="${(3*pi)/2}" />
 </robot>

File: cobot_description/urdf/sensors/ultrasoon.urdf.xacro (robot description, xacro)
@@ -5,5 +5,5 @@
     <link name="ultrasoon_${panel}_${side}_link">
        <visual>
-       <origin xyz="0 0 0" rpy="${parent_ox} ${parent_oy} ${parent_oz}" />
+       <origin xyz="0 0 0" rpy="0 0 0" />
         <geometry>
           <mesh filename="package://cobot_description/meshes/dae/ultrasoon.dae" />
