Commit message: Updated names to be the same as tf names

File: cobot_description/urdf/sensors/kinect.urdf.xacro (robot description, xacro)
@@ -2,51 +2,79 @@
 <robot name="kinect" xmlns:xacro="http://ros.org/wiki/xacro">
   <xacro:include filename="$(find cobot_description)/urdf/constants.urdf.xacro" />
-  <xacro:property name="kinect_length" value="0.275" />
-  <xacro:property name="kinect_width" value="0.05" />
-  <xacro:property name="kinect_height" value="0.055" />
-  <xacro:property name="kinect_diameter_lens" value="0.018" />
+  <xacro:property name="camera_length" value="0.275" />
+  <xacro:property name="camera_width" value="0.05" />
+  <xacro:property name="camera_height" value="0.055" />
+  <xacro:property name="camera_diameter_lens" value="0.018" />
 <xacro:macro name="kinect" params="parent_link parent_x parent_y parent_z parent_ox parent_oy parent_oz">
-  <link name="kinect_base_link">
+  <link name="camera_rgb_frame">
      <visual>
-     <origin xyz="0 0 0" rpy="${parent_ox} ${parent_oy} ${parent_oz}" />
+     <origin xyz="0 0.15 0" rpy="${parent_ox + pi/2.0} ${parent_oy} ${parent_oz}" />
       <geometry>
-        <box size="${kinect_length} ${kinect_width} ${kinect_height}" />
+        <cylinder radius="${camera_diameter_lens/2.0}" length="0.3" />
       </geometry>
-     <material name="green" />
+     <material name="black"/>
     </visual>
   </link>
-  <link name="kinect_ir_sensor_link">
+  <link name="camera_rgb_optical_frame">
      <visual>
-     <origin xyz="0 0 0" rpy="${parent_ox + pi/2.0} ${parent_oy} ${parent_oz}" />
+     <origin xyz="0 0.15 0" rpy="${parent_ox + pi/2.0} ${parent_oy} ${parent_oz}" />
       <geometry>
-        <cylinder radius="${kinect_diameter_lens/2.0}" length="1.01" />
+        <cylinder radius="${camera_diameter_lens/4.0}" length="0.3" />
       </geometry>
      <material name="white"/>
     </visual>
   </link>
-  <link name="kinect_rgb_sensor_link">
-     <visual>
-     <origin xyz="0 0 0" rpy="${parent_ox + pi/2.0} ${parent_oy} ${parent_oz}" />
+  <link name="camera_link">
+   <visual>
+    <origin xyz="0 0 0" rpy="0 0 0"/>
+     <geometry>
+       <box size="${camera_length} ${camera_width} ${camera_height}" />
+     </geometry>
+    <material name="green" />
+   </visual>
+  </link>
+	<link name="camera_depth_frame">
+   <visual>
+     <origin xyz="0 0.15 0" rpy="${parent_ox + pi/2.0} ${parent_oy} ${parent_oz}" />
       <geometry>
-        <cylinder radius="${kinect_diameter_lens/2.0}" length="1.01" />
+        <cylinder radius="${camera_diameter_lens/2.0}" length="0.3" />
       </geometry>
      <material name="black"/>
     </visual>
   </link>
-  <joint name="kinect_base_top_joint" type="fixed">
+	<link name="camera_depth_optical_frame">
+   <visual>
+     <origin xyz="0 0.15 0" rpy="${parent_ox + pi/2.0} ${parent_oy} ${parent_oz}" />
+      <geometry>
+        <cylinder radius="${camera_diameter_lens/4.0}" length="0.3" />
+      </geometry>
+     <material name="red"/>
+    </visual>
+  </link>
+  <joint name="camera_rgb_joint" type="fixed">
+    <origin xyz="${parent_x} ${parent_y} ${parent_z}" rpy="${parent_ox} ${parent_oy} ${parent_oz}" />
     <parent link="${parent_link}" />
-    <child link="kinect_base_link" />
-    <origin xyz="${parent_x} ${parent_y} ${parent_z}" rpy="${parent_ox} ${parent_oy} ${parent_oz}" />
+    <child link="camera_rgb_frame" />
   </joint>
-  <joint name="kinect_ir_sensor_kinect_base_joint" type="fixed">
-    <parent link="kinect_base_link" />
-    <child link="kinect_ir_sensor_link" />
-    <origin xyz="-0.013 0 0" rpy="0 0 0" />
-  </joint>
-  <joint name="kinect_rgb_sensor_kinect_base_joint" type="fixed">
-    <parent link="kinect_base_link" />
-    <child link="kinect_rgb_sensor_link" />
-    <origin xyz="0.013 0 0" rpy="0 0 0" />
-  </joint>
+   <joint name="camera_rgb_optical_joint" type="fixed">
+     <origin xyz="0 0 0" rpy="0 0 0" />
+     <parent link="camera_rgb_frame" />
+     <child link="camera_rgb_optical_frame" />
+   </joint>
+   <joint name="camera_joint" type="fixed">
+     <origin xyz="0.007 0 0" rpy="0 0 0"/>
+     <parent link="camera_rgb_frame"/>
+     <child link="camera_link"/>
+   </joint>
+	<joint name="camera_depth_joint" type="fixed">
+	  <origin xyz="0.025 0 0" rpy="0 0 0" />
+	  <parent link="camera_rgb_frame" />
+	  <child link="camera_depth_frame" />
+	</joint>
+	<joint name="camera_depth_optical_joint" type="fixed">
+	  <origin xyz="0 0 0" rpy="0 0 0" />
+	  <parent link="camera_depth_frame" />
+	  <child link="camera_depth_optical_frame" />
+	</joint>
 </xacro:macro>
 </robot>

Commit message: Made TF camera names easy reconfigurable

File: cobot_description/urdf/sensors/kinect.urdf.xacro (robot description, xacro)
@@ -6,6 +6,7 @@
   <xacro:property name="camera_height" value="0.055" />
   <xacro:property name="camera_diameter_lens" value="0.018" />
+  <xacro:property name="camera_name"        value="kinect" />
 <xacro:macro name="kinect" params="parent_link parent_x parent_y parent_z parent_ox parent_oy parent_oz">
-  <link name="camera_rgb_frame">
+  <link name="${camera_name}_rgb_frame">
      <visual>
      <origin xyz="0.15 0 0" rpy="${parent_ox} ${parent_oy + pi/2} ${parent_oz}" />
@@ -16,5 +17,5 @@
     </visual>
   </link>
-  <link name="camera_rgb_optical_frame">
+  <link name="${camera_name}_rgb_optical_frame">
      <visual>
      <origin xyz="0.15 0 0" rpy="${parent_ox} ${parent_oy + pi/2} ${parent_oz}" />
@@ -25,5 +26,5 @@
     </visual>
   </link>
-  <link name="camera_link">
+  <link name="${camera_name}_link">
    <visual>
     <origin xyz="0 0 0" rpy="0 0 0"/>
@@ -34,5 +35,5 @@
    </visual>
   </link>
-	<link name="camera_depth_frame">
+	<link name="${camera_name}_depth_frame">
    <visual>
      <origin xyz="0.15 0 0" rpy="${parent_ox} ${parent_oy + pi/2.0} ${parent_oz}" />
@@ -43,5 +44,5 @@
     </visual>
   </link>
-	<link name="camera_depth_optical_frame">
+	<link name="${camera_name}_depth_optical_frame">
    <visual>
      <origin xyz="0.15 0 0" rpy="${parent_ox} ${parent_oy + pi/2.0} ${parent_oz}" />
@@ -52,28 +53,28 @@
     </visual>
   </link>
-  <joint name="camera_rgb_joint" type="fixed">
+  <joint name="${camera_name}_rgb_joint" type="fixed">
     <origin xyz="${parent_x} ${parent_y} ${parent_z}" rpy="${parent_ox} ${parent_oy} ${parent_oz}" />
     <parent link="${parent_link}" />
-    <child link="camera_rgb_frame" />
+    <child link="${camera_name}_rgb_frame" />
   </joint>
-   <joint name="camera_rgb_optical_joint" type="fixed">
+   <joint name="${camera_name}_rgb_optical_joint" type="fixed">
      <origin xyz="0 0 0" rpy="0 0 0" />
-     <parent link="camera_rgb_frame" />
-     <child link="camera_rgb_optical_frame" />
+     <parent link="${camera_name}_rgb_frame" />
+     <child link="${camera_name}_rgb_optical_frame" />
    </joint>
-   <joint name="camera_joint" type="fixed">
+   <joint name="${camera_name}_joint" type="fixed">
      <origin xyz="0 0.0125 0" rpy="0 0 0"/>
-     <parent link="camera_rgb_frame"/>
-     <child link="camera_link"/>
+     <parent link="${camera_name}_rgb_frame"/>
+     <child link="${camera_name}_link"/>
    </joint>
-	<joint name="camera_depth_joint" type="fixed">
+	<joint name="${camera_name}_depth_joint" type="fixed">
 	  <origin xyz="0 0.027 0" rpy="0 0 0" />
-	  <parent link="camera_rgb_frame" />
-	  <child link="camera_depth_frame" />
+	  <parent link="${camera_name}_rgb_frame" />
+	  <child link="${camera_name}_depth_frame" />
 	</joint>
-	<joint name="camera_depth_optical_joint" type="fixed">
+	<joint name="${camera_name}_depth_optical_joint" type="fixed">
 	  <origin xyz="0 0 0" rpy="0 0 0" />
-	  <parent link="camera_depth_frame" />
-	  <child link="camera_depth_optical_frame" />
+	  <parent link="${camera_name}_depth_frame" />
+	  <child link="${camera_name}_depth_optical_frame" />
 	</joint>
 </xacro:macro>
